File: Hardware/sparkfun-atsamd21g-breakout.sch (EAGLE design)
At the start: 41 parts, among them Q1 2N7002PW, Q3 2.5A/30V, U1 ATSAMD21G-A, U2 MIC5219 3.3V, U4 74AHC1G125

Commit message: Minor, pre-checklist modifications.
Parts:
- C5, C6: value 22pF -> 15pF; device SparkFun-Capacitors:CAP0402-CAP -> samd21-temp:15PF-50V(+-5%)(0402)
- D1: value Yellow -> GREEN; device SparkFun-LED:LED-YELLOW0603 -> SparkFun-LED:LED-GREEN0603
- D4: value GREEN -> Yellow; device SparkFun-LED:LED-GREEN0603 -> SparkFun-LED:LED-YELLOW0603
- Y1: value (none) -> 32.768kHz
Other:
- note added: "ATSAMD21G18 VDD Range: 1.62-3.63V"
- note added: "SJ1 enable's disconnecting the Power LED indicator. For power-saving requirements. Default: closed."
- moved on the sheet: C1, D1, D2, D3, D4, Q1, R2, R3, R6, R8, SJ1

Commit message: Adding PROD_ID's to new parts.
Parts:
- L1: PROD_ID (none) -> RES-07859
Changed lines of the file:
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@@
 <part name="GND2" library="SparkFun-Aesthetics" deviceset="GND" device=""/>
 <part name="GND3" library="SparkFun-Aesthetics" deviceset="GND" device=""/>
-<part name="L1" library="SparkFun-Passives" deviceset="INDUCTOR" device="0603" value="FB - 30Ohm"/>
+<part name="L1" library="SparkFun-Passives" deviceset="INDUCTOR" device="0603" value="FB - 30Ohm">
+<attribute name="PROD_ID" value="RES-07859"/>
+</part>
 <part name="GND4" library="SparkFun-Aesthetics" deviceset="GND" device=""/>
 <part name="SUPPLY3" library="SparkFun-Aesthetics" deviceset="3.3V" device=""/>
@@
 <attribute name="NAME" x="17.78" y="88.9" size="1.778" layer="95"/>
 <attribute name="VALUE" x="14.224" y="76.2" size="1.778" layer="96" rot="R90"/>
+<attribute name="PROD_ID" x="15.24" y="83.82" size="1.27" layer="96" align="center-left" display="off"/>
 </instance>
 <instance part="GND4" gate="1" x="15.24" y="58.42"/>

Commit message: Renaming U4 to U3, adding tSilk to pin 11, dimension to .008in.
Parts:
- removed U4: 74AHC1G125, SparkFun-DigitalIC:74AHC1G125
- added JP3: (no value), SparkFun-Connectors:USB-ABCONN-11794
- U3: value (none) -> 74AHC1G125; device SparkFun-Connectors:USB-ABCONN-11794 -> SparkFun-DigitalIC:74AHC1G125
Connections:
- net 3.3V: now also U3.VCC; no longer U4.VCC
- net GND: now also JP3.GND, JP3.SHIELD; no longer U3.SHIELD, U4.GND
- net N$1: now also JP3.VBUS; no longer U3.VBUS
- net N$8: now also JP3.USBID, U3./OE, U3.A; no longer U3.USBID, U4./OE, U4.A
- net N$9: now also U3.Y; no longer U4.Y
- net USB_D+: now also JP3.D+; no longer U3.D+
- net USB_D-: now also JP3.D-; no longer U3.D-
Changed lines of the file:
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@@
 <part name="JP4" library="SparkFun-Connectors" deviceset="M02" device="1X02_NO_SILK"/>
 <part name="F1" library="SparkFun-PowerIC" deviceset="PTC" device="SMD" value="500mA"/>
-<part name="U3" library="SparkFun-Connectors" deviceset="USB-AB" device="CONN-11794"/>
-<part name="U4" library="SparkFun-DigitalIC" deviceset="74AHC1G125" device=""/>
+<part name="JP3" library="SparkFun-Connectors" deviceset="USB-AB" device="CONN-11794"/>
+<part name="U3" library="SparkFun-DigitalIC" deviceset="74AHC1G125" device=""/>
 <part name="R4" library="SparkFun-Resistors" deviceset="100KOHM-1/10W-1%(0603)" device="" value="100k"/>
 <part name="SUPPLY10" library="SparkFun-Aesthetics" deviceset="3.3V" device=""/>
@@
 <instance part="JP4" gate="G$1" x="228.6" y="60.96"/>
 <instance part="F1" gate="G$1" x="50.8" y="167.64"/>
-<instance part="U3" gate="G$1" x="22.86" y="162.56" rot="R180"/>
-<instance part="U4" gate="G$1" x="66.04" y="134.62"/>
+<instance part="JP3" gate="G$1" x="22.86" y="162.56" rot="R180"/>
+<instance part="U3" gate="G$1" x="66.04" y="134.62"/>
 <instance part="R4" gate="G$1" x="43.18" y="144.78" rot="R90"/>
 <instance part="SUPPLY10" gate="G$1" x="43.18" y="152.4"/>
@@
 <wire x1="27.94" y1="157.48" x2="30.48" y2="157.48" width="0.1524" layer="91"/>
 <wire x1="30.48" y1="157.48" x2="30.48" y2="152.4" width="0.1524" layer="91"/>
-<pinref part="U3" gate="G$1" pin="GND"/>
-<pinref part="U3" gate="G$1" pin="SHIELD"/>
+<pinref part="JP3" gate="G$1" pin="GND"/>
+<pinref part="JP3" gate="G$1" pin="SHIELD"/>
 <wire x1="27.94" y1="170.18" x2="30.48" y2="170.18" width="0.1524" layer="91"/>
 <wire x1="30.48" y1="170.18" x2="30.48" y2="157.48" width="0.1524" layer="91"/>
@@
 </segment>
 <segment>
-<pinref part="U4" gate="G$1" pin="GND"/>
+<pinref part="U3" gate="G$1" pin="GND"/>
 <pinref part="GND7" gate="1" pin="GND"/>
 <wire x1="53.34" y1="132.08" x2="50.8" y2="132.08" width="0.1524" layer="91"/>
@@
 </segment>
 <segment>
-<pinref part="U4" gate="G$1" pin="VCC"/>
+<pinref part="U3" gate="G$1" pin="VCC"/>
 <pinref part="SUPPLY11" gate="G$1" pin="3.3V"/>
 <wire x1="78.74" y1="137.16" x2="81.28" y2="137.16" width="0.1524" layer="91"/>
@@
 <wire x1="27.94" y1="162.56" x2="35.56" y2="162.56" width="0.1524" layer="91"/>
 <label x="35.56" y="162.56" size="1.27" layer="95" xref="yes"/>
-<pinref part="U3" gate="G$1" pin="D+"/>
+<pinref part="JP3" gate="G$1" pin="D+"/>
 </segment>
 </net>
@@
 <wire x1="27.94" y1="165.1" x2="35.56" y2="165.1" width="0.1524" layer="91"/>
 <label x="35.56" y="165.1" size="1.27" layer="95" xref="yes"/>
-<pinref part="U3" gate="G$1" pin="D-"/>
+<pinref part="JP3" gate="G$1" pin="D-"/>
 </segment>
 </net>
@@
 <pinref part="F1" gate="G$1" pin="1"/>
 <wire x1="45.72" y1="167.64" x2="27.94" y2="167.64" width="0.1524" layer="91"/>
-<pinref part="U3" gate="G$1" pin="VBUS"/>
+<pinref part="JP3" gate="G$1" pin="VBUS"/>
 </segment>
 </net>
@@
 <net name="N$8" class="0">
 <segment>
-<pinref part="U4" gate="G$1" pin="/OE"/>
+<pinref part="U3" gate="G$1" pin="/OE"/>
 <wire x1="53.34" y1="137.16" x2="50.8" y2="137.16" width="0.1524" layer="91"/>
-<pinref part="U4" gate="G$1" pin="A"/>
+<pinref part="U3" gate="G$1" pin="A"/>
 <wire x1="50.8" y1="137.16" x2="48.26" y2="137.16" width="0.1524" layer="91"/>
 <wire x1="48.26" y1="137.16" x2="43.18" y2="137.16" width="0.1524" layer="91"/>
@@
 <junction x="48.26" y="137.16"/>
 <wire x1="48.26" y1="137.16" x2="48.26" y2="160.02" width="0.1524" layer="91"/>
-<pinref part="U3" gate="G$1" pin="USBID"/>
+<pinref part="JP3" gate="G$1" pin="USBID"/>
 <wire x1="48.26" y1="160.02" x2="27.94" y2="160.02" width="0.1524" layer="91"/>
 </segment>
@@
 <net name="N$9" class="0">
 <segment>
-<pinref part="U4" gate="G$1" pin="Y"/>
+<pinref part="U3" gate="G$1" pin="Y"/>
 <pinref part="Q3" gate="G$1" pin="G"/>
 <wire x1="78.74" y1="132.08" x2="83.82" y2="132.08" width="0.1524" layer="91"/>

Commit message: Moving silk. Swapping D4 and D2.
Connections:
- net D2: now also U1.PA14(XIN/SER2:2+); no longer U1.PA08(I2C/AIN16/SER0:0+)
- net D4: now also U1.PA08(I2C/AIN16/SER0:0+); no longer U1.PA14(XIN/SER2:2+)
Other:
- note added: "v10"
- note removed: "v01"
Changed lines of the file:
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@@
 <text x="2.54" y="119.38" size="2.54" layer="94" align="top-left">ATSAMD21G</text>
 <text x="170.18" y="10.16" size="2.54" layer="94" align="top-left">Jim Lindblom</text>
-<text x="238.76" y="10.16" size="2.54" layer="94" align="top-left">v01</text>
+<text x="238.76" y="10.16" size="2.54" layer="94" align="top-left">v10</text>
 <text x="48.26" y="106.68" size="1.778" layer="97" align="center-left">ATSAMD21G18
 VDD Range: 1.62-3.63V</text>
@@
 </segment>
 </net>
+<net name="D4" class="0">
+<segment>
+<pinref part="U1" gate="G$1" pin="PA08(I2C/AIN16/SER0:0+)"/>
+<wire x1="111.76" y1="88.9" x2="114.3" y2="88.9" width="0.1524" layer="91"/>
+<label x="114.3" y="88.9" size="1.27" layer="95" xref="yes"/>
+</segment>
+<segment>
+<pinref part="JP1" gate="G$1" pin="6"/>
+<wire x1="175.26" y1="63.5" x2="180.34" y2="63.5" width="0.1524" layer="91"/>
+<label x="180.34" y="63.5" size="1.27" layer="95" xref="yes"/>
+</segment>
+</net>
+<net name="D3" class="0">
+<segment>
+<pinref part="JP1" gate="G$1" pin="7"/>
+<wire x1="175.26" y1="66.04" x2="180.34" y2="66.04" width="0.1524" layer="91"/>
+<label x="180.34" y="66.04" size="1.27" layer="95" xref="yes"/>
+</segment>
+<segment>
+<pinref part="U1" gate="G$1" pin="PA09(I2C/AIN17/SER0:1+)"/>
+<wire x1="111.76" y1="86.36" x2="114.3" y2="86.36" width="0.1524" layer="91"/>
+<label x="114.3" y="86.36" size="1.27" layer="95" xref="yes"/>
+</segment>
+</net>
 <net name="D2" class="0">
+<segment>
+<pinref part="U1" gate="G$1" pin="PA14(XIN/SER2:2+)"/>
+<wire x1="111.76" y1="73.66" x2="114.3" y2="73.66" width="0.1524" layer="91"/>
+<label x="114.3" y="73.66" size="1.27" layer="95" xref="yes"/>
+</segment>
 <segment>
 <pinref part="JP1" gate="G$1" pin="8"/>
@@
 <label x="180.34" y="68.58" size="1.27" layer="95" xref="yes"/>
 </segment>
-<segment>
-<pinref part="U1" gate="G$1" pin="PA08(I2C/AIN16/SER0:0+)"/>
-<wire x1="111.76" y1="88.9" x2="114.3" y2="88.9" width="0.1524" layer="91"/>
-<label x="114.3" y="88.9" size="1.27" layer="95" xref="yes"/>
-</segment>
-</net>
-<net name="D3" class="0">
-<segment>
-<pinref part="JP1" gate="G$1" pin="7"/>
-<wire x1="175.26" y1="66.04" x2="180.34" y2="66.04" width="0.1524" layer="91"/>
-<label x="180.34" y="66.04" size="1.27" layer="95" xref="yes"/>
-</segment>
-<segment>
-<pinref part="U1" gate="G$1" pin="PA09(I2C/AIN17/SER0:1+)"/>
-<wire x1="111.76" y1="86.36" x2="114.3" y2="86.36" width="0.1524" layer="91"/>
-<label x="114.3" y="86.36" size="1.27" layer="95" xref="yes"/>
-</segment>
-</net>
-<net name="D4" class="0">
-<segment>
-<pinref part="JP1" gate="G$1" pin="6"/>
-<wire x1="175.26" y1="63.5" x2="180.34" y2="63.5" width="0.1524" layer="91"/>
-<label x="180.34" y="63.5" size="1.27" layer="95" xref="yes"/>
-</segment>
-<segment>
-<pinref part="U1" gate="G$1" pin="PA14(XIN/SER2:2+)"/>
-<wire x1="111.76" y1="73.66" x2="114.3" y2="73.66" width="0.1524" layer="91"/>
-<label x="114.3" y="73.66" size="1.27" layer="95" xref="yes"/>
-</segment>
-</net>
+</net>

Commit message: Pulling buffer power up to RAW
Connections:
- net 3.3V: no longer R4.2, U3.VCC
- net RAW: now also R4.2, U3.VCC
Changed lines of the file:
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@@
 <part name="U3" library="SparkFun-DigitalIC" deviceset="74AHC1G125" device=""/>
 <part name="R4" library="SparkFun-Resistors" deviceset="100KOHM-1/10W-1%(0603)" device="" value="100k"/>
-<part name="SUPPLY10" library="SparkFun-Aesthetics" deviceset="3.3V" device=""/>
-<part name="SUPPLY11" library="SparkFun-Aesthetics" deviceset="3.3V" device=""/>
 <part name="GND7" library="SparkFun-Aesthetics" deviceset="GND" device=""/>
 <part name="R5" library="SparkFun-Resistors" deviceset="330OHM1/10W1%(0603)" device="" value="330"/>
@@
 <instance part="U3" gate="G$1" x="66.04" y="134.62"/>
 <instance part="R4" gate="G$1" x="43.18" y="144.78" rot="R90"/>
-<instance part="SUPPLY10" gate="G$1" x="43.18" y="152.4"/>
-<instance part="SUPPLY11" gate="G$1" x="81.28" y="142.24"/>
 <instance part="GND7" gate="1" x="50.8" y="127"/>
 <instance part="R5" gate="G$1" x="35.56" y="137.16"/>
@@
 </segment>
 <segment>
-<pinref part="R4" gate="G$1" pin="2"/>
-<pinref part="SUPPLY10" gate="G$1" pin="3.3V"/>
-<wire x1="43.18" y1="152.4" x2="43.18" y2="149.86" width="0.1524" layer="91"/>
-</segment>
-<segment>
-<pinref part="U3" gate="G$1" pin="VCC"/>
-<pinref part="SUPPLY11" gate="G$1" pin="3.3V"/>
-<wire x1="78.74" y1="137.16" x2="81.28" y2="137.16" width="0.1524" layer="91"/>
-<wire x1="81.28" y1="137.16" x2="81.28" y2="142.24" width="0.1524" layer="91"/>
-</segment>
-<segment>
 <pinref part="R6" gate="G$1" pin="2"/>
 <pinref part="SUPPLY12" gate="G$1" pin="3.3V"/>
@@
 <pinref part="R7" gate="G$1" pin="2"/>
 </segment>
-</net>
+<segment>
+<pinref part="U3" gate="G$1" pin="VCC"/>
+<wire x1="78.74" y1="137.16" x2="81.28" y2="137.16" width="0.1524" layer="91"/>
+<wire x1="81.28" y1="137.16" x2="81.28" y2="152.4" width="0.1524" layer="91"/>
+<label x="78.74" y="152.4" size="1.27" layer="95" rot="R180" xref="yes"/>
+<wire x1="81.28" y1="152.4" x2="78.74" y2="152.4" width="0.1524" layer="91"/>
+</segment>
+<segment>
+<pinref part="R4" gate="G$1" pin="2"/>
+<wire x1="43.18" y1="149.86" x2="43.18" y2="152.4" width="0.1524" layer="91"/>
+<wire x1="43.18" y1="152.4" x2="40.64" y2="152.4" width="0.1524" layer="91"/>
+<label x="40.64" y="152.4" size="1.27" layer="95" rot="R180" xref="yes"/>
+</segment>
+</net>
